File: gsw141-breakout/gsw141-breakout.kicad_sch (KiCad schematic)
At the start: 97 parts, among them IC1 TPS564247DRLR, IC2 TPS564247DRLR, J1 1149848, J3 HSEC8-109-01-L-RA-TR, J4 Barrel_Jack_Switch, J6 Conn_01x08, J7 Conn_01x08, SW1 SW_DIP_x09, SW2 PB400EEQR1BLK, Y1 Crystal_GND24

Commit message: latest updates to the GSW breakout
Parts:
- removed IC2: TPS564247DRLR, local:SOTFL50P160X60-6N, symbol TPS564247DRLR:TPS564247DRLR
- added C24, C25, C26, C27, C28, C29, C30, C31, C32, C33, C34, C35, C36, C37, C38, C39, C40, C41, C42, C43, C44, C45: 100n, Capacitor_SMD:C_0805_2012Metric_Pad1.18x1.45mm_HandSolder, symbol Device:C_Small
- added IC2: TPS563207DRLR, local:SOTFL50P160X60-6N, symbol TPS563207DRLR:TPS563207DRLR
- C15: value 22u -> 47u
- L1: value 1.5uH -> 2.2uH; footprint Inductor_SMD:L_0805_2012Metric_Pad1.15x1.40mm_HandSolder -> Inductor_SMD:L_Abracon_ASPI-0425
- L2: value 1uH -> 2.2uH; footprint Inductor_SMD:L_0805_2012Metric_Pad1.15x1.40mm_HandSolder -> Inductor_SMD:L_Abracon_ASPI-0425
- R31: value 8k -> 16k
Connections:
- net +1V1: now also C35.2, C36.2, C37.2, C38.2, C39.2, C40.2, C41.2, C42.2, C43.2, C44.2; no longer C15.2, C16.2, C18.2, L2.2, R31.1
- net +3.3V: now also C18.2, C24.2, C25.2, C26.2, C27.2, C28.2, C29.2, C30.2, C31.2, C32.2, C33.2, C34.2
- net A0+: now also J1.D1; no longer J1.A1
- net A0-: now also J1.D2; no longer J1.A2
- net A1+: now also J1.D3; no longer J1.A3
- net A1-: now also J1.D4; no longer J1.A4
- net A2+: now also J1.D5; no longer J1.A5
- net A2-: now also J1.D6; no longer J1.A6
- net A3+: now also J1.D7; no longer J1.A7
- net A3-: now also J1.D8; no longer J1.A8
- net B0+: now also J1.C1; no longer J1.B1
- net B0-: now also J1.C2; no longer J1.B2
- net B1+: now also J1.C3; no longer J1.B3
- net B1-: now also J1.C4; no longer J1.B4
- net B2+: now also J1.C5; no longer J1.B5
- net B2-: now also J1.C6; no longer J1.B6
- net B3+: now also J1.C7; no longer J1.B7
- net B3-: now also J1.C8; no longer J1.B8
- net C0+: now also J1.B1; no longer J1.C1
- net C0-: now also J1.B2; no longer J1.C2
- net C1+: now also J1.B3; no longer J1.C3
- net C1-: now also J1.B4; no longer J1.C4
- net C2+: now also J1.B5; no longer J1.C5
- net C2-: now also J1.B6; no longer J1.C6
- net C3+: now also J1.B7; no longer J1.C7
- net C3-: now also J1.B8; no longer J1.C8
- net D0+: now also J1.A1; no longer J1.D1
- net D0-: now also J1.A2; no longer J1.D2
- net D1+: now also J1.A3; no longer J1.D3
- net D1-: now also J1.A4; no longer J1.D4
- net D2+: now also J1.A5; no longer J1.D5
- net D2-: now also J1.A6; no longer J1.D6
- net D3+: now also J1.A7; no longer J1.D7
- net D3-: now also J1.A8; no longer J1.D8
- net FB2: now also IC2.6 (FB)
- net GND: now also C24.1, C25.1, C26.1, C27.1, C28.1, C29.1, C30.1, C31.1, C32.1, C33.1, C34.1, C35.1, C36.1, C37.1, C38.1, C39.1, C40.1, C41.1, C42.1, C43.1, C44.1, IC2.3 (GND)
- net LED0L: now also J1.D10 (K_GREEN_4); no longer J1.A10 (K_GREEN_1)
- net LED0R: now also J1.D12 (K_YELLOW_4); no longer J1.A12 (K_YELLOW_1)
- net LED1L: now also J1.C10 (K_GREEN_3); no longer J1.B10 (K_GREEN_2)
- net LED1R: now also J1.C12 (K_YELLOW_3); no longer J1.B12 (K_YELLOW_2)
- net LED2L: now also J1.B10 (K_GREEN_2); no longer J1.C10 (K_GREEN_3)
- net LED2R: now also J1.B12 (K_YELLOW_2); no longer J1.C12 (K_YELLOW_3)
- net LED3L: now also J1.A10 (K_GREEN_1); no longer J1.D10 (K_GREEN_4)
- net LED3R: now also J1.A12 (K_YELLOW_1); no longer J1.D12 (K_YELLOW_4)
- net PWR_EN2: now also IC2.5 (EN)
- net PWR_UNREG: now also IC2.1 (VIN)
- net SW2: now also C45.2, IC2.2 (SW)
- new net: C45.1, IC2.4 (BST)
- new net NOISY_LOWV: C15.2, C16.2, L2.2, R31.1
- no-connect marks 2 -> 3
Other:
- moved on the sheet: C17
