File: gsw141-breakout/gsw141-breakout.kicad_pcb (KiCad board)
At the start: 4 copper layers, 86.7 x 96 mm, 97 parts, among them IC1 TPS564247DRLR, IC2 TPS564247DRLR, J1 1149848, J3 HSEC8-109-01-L-RA-TR, J4 Barrel_Jack_Switch, J6 Conn_01x08, J7 Conn_01x08, SW1 SW_DIP_x09, SW2 PB400EEQR1BLK, Y1 Crystal_GND24

Commit message: latest updates to the GSW breakout
Parts:
- added C24: 100n, Capacitor_SMD:C_0805_2012Metric_Pad1.18x1.45mm_HandSolder, B.Cu at (174.9, 102.8)
- added C25: 100n, Capacitor_SMD:C_0805_2012Metric_Pad1.18x1.45mm_HandSolder, B.Cu at (175.0, 105.0)
- added C26: 100n, Capacitor_SMD:C_0805_2012Metric_Pad1.18x1.45mm_HandSolder, B.Cu at (174.9, 86.9)
- added C27: 100n, Capacitor_SMD:C_0805_2012Metric_Pad1.18x1.45mm_HandSolder, B.Cu at (175.0, 89.1)
- added C28: 100n, Capacitor_SMD:C_0805_2012Metric_Pad1.18x1.45mm_HandSolder, B.Cu at (175.0, 91.3)
- added C29: 100n, Capacitor_SMD:C_0805_2012Metric_Pad1.18x1.45mm_HandSolder, B.Cu at (170.4, 101.3)
- added C30: 100n, Capacitor_SMD:C_0805_2012Metric_Pad1.18x1.45mm_HandSolder, B.Cu at (168.0, 101.3)
- added C31: 100n, Capacitor_SMD:C_0805_2012Metric_Pad1.18x1.45mm_HandSolder, B.Cu at (165.7, 101.3)
- added C32: 100n, Capacitor_SMD:C_0805_2012Metric_Pad1.18x1.45mm_HandSolder, B.Cu at (163.3, 101.3)
- added C33: 100n, Capacitor_SMD:C_0805_2012Metric_Pad1.18x1.45mm_HandSolder, B.Cu at (160.9, 101.3)
- added C34: 100n, Capacitor_SMD:C_0805_2012Metric_Pad1.18x1.45mm_HandSolder, B.Cu at (158.5, 101.3)
- added C35: 100n, Capacitor_SMD:C_0805_2012Metric_Pad1.18x1.45mm_HandSolder, B.Cu at (168.3, 88.2)
- added C36: 100n, Capacitor_SMD:C_0805_2012Metric_Pad1.18x1.45mm_HandSolder, B.Cu at (162.0, 97.0)
- added C37: 100n, Capacitor_SMD:C_0805_2012Metric_Pad1.18x1.45mm_HandSolder, B.Cu at (175.0, 96.3)
- added C38: 100n, Capacitor_SMD:C_0805_2012Metric_Pad1.18x1.45mm_HandSolder, B.Cu at (175.0, 98.4)
- added C39: 100n, Capacitor_SMD:C_0805_2012Metric_Pad1.18x1.45mm_HandSolder, B.Cu at (170.8, 88.3)
- added C40: 100n, Capacitor_SMD:C_0805_2012Metric_Pad1.18x1.45mm_HandSolder, B.Cu at (175.0, 93.4)
- added C41: 100n, Capacitor_SMD:C_0805_2012Metric_Pad1.18x1.45mm_HandSolder, B.Cu at (166.0, 88.2)
- added C42: 100n, Capacitor_SMD:C_0805_2012Metric_Pad1.18x1.45mm_HandSolder, B.Cu at (162.0, 92.0)
- added C43: 100n, Capacitor_SMD:C_0805_2012Metric_Pad1.18x1.45mm_HandSolder, B.Cu at (163.6, 88.3)
- added C44: 100n, Capacitor_SMD:C_0805_2012Metric_Pad1.18x1.45mm_HandSolder, B.Cu at (162.0, 94.5)
- added C45: 100n, Capacitor_SMD:C_0805_2012Metric_Pad1.18x1.45mm_HandSolder, F.Cu at (177.6, 119.3)
- C15: value 22u -> 47u
- IC2: value TPS564247DRLR -> TPS563207DRLR
- J1, J4, J6, J7, SW1, SW2: moved to B.Cu
- L1: value 1.5uH -> 2.2uH; footprint Inductor_SMD:L_0805_2012Metric_Pad1.15x1.40mm_HandSolder -> Inductor_SMD:L_Abracon_ASPI-0425
- L2: value 1uH -> 2.2uH; footprint Inductor_SMD:L_0805_2012Metric_Pad1.15x1.40mm_HandSolder -> Inductor_SMD:L_Abracon_ASPI-0425
- R1, R2, R27, R28, R30: moved to F.Cu
- R31: value 8k -> 16k
- moved R28 60.1 mm to (121.9, 58.5)
- moved R1 57.9 mm to (123.9, 125.6)
- moved R27 40.5 mm to (116.4, 74.8)
- moved R2 39.7 mm to (116.8, 109.1), turned to 0 degrees
- moved J1 39.4 mm to (116.3, 112.5), turned to 90 degrees
- moved R25 20.7 mm to (116.8, 106.6), turned to 180 degrees
- moved R30 20.6 mm to (116.4, 78.5), turned to 0 degrees
- moved C18 13.3 mm to (175.0, 100.6), turned to 180 degrees
- moved C17 12.2 mm to (156.1, 101.3)
- moved R51 10.2 mm to (160.7, 89.6)
- moved R34 6.97 mm to (169.8, 132.3)
- moved R35 6.97 mm to (172.3, 132.3)
- moved R37 6.97 mm to (174.9, 132.3)
- moved R39 6.97 mm to (177.4, 132.3)
- moved R41 6.97 mm to (180.0, 132.3)
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Connections:
- C15 pad 2: +1V1 -> /NOISY_LOWV
- C16 pad 2: +1V1 -> /NOISY_LOWV
- C18 pad 2: +1V1 -> +3.3V
- IC2 pad 4: GND -> Net-(IC2-BST)
- J1 pad A1: /A0+ -> /D0+
- J1 pad A10: /LED0L -> /LED3L
- J1 pad A12: /LED0R -> /LED3R
- J1 pad A2: /A0- -> /D0-
- J1 pad A3: /A1+ -> /D1+
- J1 pad A4: /A1- -> /D1-
- J1 pad A5: /A2+ -> /D2+
- J1 pad A6: /A2- -> /D2-
- J1 pad A7: /A3+ -> /D3+
- J1 pad A8: /A3- -> /D3-
- J1 pad B1: /B0+ -> /C0+
- J1 pad B10: /LED1L -> /LED2L
- J1 pad B12: /LED1R -> /LED2R
- J1 pad B2: /B0- -> /C0-
- J1 pad B3: /B1+ -> /C1+
- J1 pad B4: /B1- -> /C1-
- J1 pad B5: /B2+ -> /C2+
- J1 pad B6: /B2- -> /C2-
- J1 pad B7: /B3+ -> /C3+
- J1 pad B8: /B3- -> /C3-
- J1 pad C1: /C0+ -> /B0+
- J1 pad C10: /LED2L -> /LED1L
- J1 pad C12: /LED2R -> /LED1R
- J1 pad C2: /C0- -> /B0-
- J1 pad C3: /C1+ -> /B1+
- J1 pad C4: /C1- -> /B1-
- J1 pad C5: /C2+ -> /B2+
- J1 pad C6: /C2- -> /B2-
- J1 pad C7: /C3+ -> /B3+
- J1 pad C8: /C3- -> /B3-
- J1 pad D1: /D0+ -> /A0+
- J1 pad D10: /LED3L -> /LED0L
- J1 pad D12: /LED3R -> /LED0R
- J1 pad D2: /D0- -> /A0-
- J1 pad D3: /D1+ -> /A1+
- J1 pad D4: /D1- -> /A1-
- J1 pad D5: /D2+ -> /A2+
- J1 pad D6: /D2- -> /A2-
- J1 pad D7: /D3+ -> /A3+
- J1 pad D8: /D3- -> /A3-
- L2 pad 2: +1V1 -> /NOISY_LOWV
- R31 pad 1: +1V1 -> /NOISY_LOWV
Routing:
- net Earth: track 138.6 -> 0.00 mm
- net +3.3V: track 296.9 -> 213.1 mm, vias 14 -> 10
- net /LED3R: track 58.1 -> 0.00 mm, vias 1 -> 0
- net /GPIO28: track 80.2 -> 24.3 mm, vias 1 -> 0
- net /LED3L: track 50.5 -> 0.00 mm, vias 1 -> 0
- net /MSCK: track 55.4 -> 6.91 mm, vias 2 -> 0
- net /UART_TX: track 53.7 -> 10.6 mm, vias 2 -> 0
- net /SMDC: track 39.5 -> 0.00 mm, vias 1 -> 0
- net /UART_RX: track 39.0 -> 0.00 mm, vias 1 -> 0
- net /GPIO00: track 38.6 -> 0.00 mm, vias 2 -> 0
- net /PWR_UNREG: track 81.5 -> 44.5 mm
- net /SMDIO: track 36.1 -> 0.00 mm, vias 1 -> 0
- net /GPIO29: track 59.7 -> 24.1 mm, vias 1 -> 0
- net /MSD0: track 48.4 -> 12.8 mm, vias 2 -> 0
- net /MSCS: track 50.2 -> 14.9 mm, vias 2 -> 0
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- removed copper zone on B.Cu, net GND
- removed copper zone on F.Cu, net GND
