File: SYZYGY-RGMII-tester/SYZYGY-RGMII-tester.kicad_pcb (KiCad board)
At the start: 4 copper layers, 27.6 x 28.4 mm, 6 parts, among them J1 Conn_02x07_Odd_Even, J2 Conn_01x02, J3 QSH-020-01-X-D-DP-A, J4 Conn_02x06_Odd_Even

Commit message: mild board updates before ordering
Parts:
- moved J2 1.42 mm to (111.9, 96.2)
Other:
- board text added: "Lo | Hi"
- board text added: "RGMII over SYZYGY Test Board @rustbox rev2 2024-10-02"
- board text removed: "Hi | Lo"
- board text removed: "RGMII over SYZYGY Test Board @rustbox rev1 2024-08-30"
Changed lines of the file:
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@@
 	(footprint "Connector_PinHeader_2.54mm:PinHeader_1x02_P2.54mm_Horizontal"
 		(layer "B.Cu")
-		(at 110.5 96.2 180)
+		(at 111.92 96.2 180)
 		(descr "Through hole angled pin header, 1x02, 2.54mm pitch, 6mm pin length, single row")
 		(tags "Through hole angled pin header THT 1x02 2.54mm single row")
 		(property "Reference" "J2"
-			(at 5.1 0 360)
+			(at 5.1 0 0)
 			(layer "B.SilkS")
 			(effects
@@
 		)
 		(property "Value" "Conn_01x02"
-			(at 4.385 -4.81 360)
+			(at 4.385 -4.81 0)
 			(layer "B.Fab")
 			(effects
@@
 		(tags "Through hole pin header THT 2x07 2.54mm double row")
 		(property "Reference" "J1"
-			(at 0 2.1 360)
+			(at 0 2.1 0)
 			(layer "B.SilkS")
 			(effects
@@
 		)
 		(property "Value" "Conn_02x07_Odd_Even"
-			(at 1.27 -17.57 360)
+			(at 1.27 -17.57 0)
 			(layer "B.Fab")
 			(effects
@@
 		(tags "Through hole pin header THT 2x06 2.54mm double row")
 		(property "Reference" "J4"
-			(at 2.54 -14.9 90)
+			(at 5.34 -14.95 90)
 			(layer "B.SilkS")
 			(effects
@@
 		)
 		(fp_text user "${REFERENCE}"
-			(at 1.27 -6.35 360)
+			(at 1.27 -6.35 0)
 			(layer "B.Fab")
 			(effects
@@
 		(start 114.5 99.2)
 		(end 114.7 99.2)
+		(stroke
+			(width 0.1)
+			(type default)
+		)
+		(layer "B.SilkS")
+	)
+	(gr_line
+		(start 115.4 97.45)
+		(end 113.8 97.45)
 		(stroke
 			(width 0.1)
@@
 		)
 	)
-	(gr_text "Hi | Lo  "
-		(at 108.8 93.1 0)
+	(gr_text "Lo | Hi  "
+		(at 108.95 93.45 0)
 		(layer "B.SilkS")
 		(effects
@@
 		)
 	)
-	(gr_text "RGMII over SYZYGY\nTest Board\n@rustbox\nrev1 2024-08-30"
+	(gr_text "RGMII over SYZYGY\nTest Board\n@rustbox\nrev2 2024-10-02"
 		(at 130 83.7 0)
 		(layer "B.SilkS")
@@
 	)
 	(gr_text "GND"
-		(at 113.5 95 90)
+		(at 110.1 93.3 180)
 		(layer "B.SilkS")
 		(effects
